Commit message: adding indoor code

File: build/vrx/wamv_gazebo/urdf/wamv_gazebo.urdf (robot description, URDF)
Before this commit: robot WAM-V, 8 links, 7 joints
Joints:
- joint wamv/left_chasis_engine_joint: limit lower=-3.14159265359 upper=3.14159265359 effort=10 velocity=10 -> lower=-3.141592653589793 upper=3.141592653589793 effort=10 velocity=10
- joint wamv/right_chasis_engine_joint: limit lower=-3.14159265359 upper=3.14159265359 effort=10 velocity=10 -> lower=-3.141592653589793 upper=3.141592653589793 effort=10 velocity=10
